File: pcb/MicroSD/MicroSD.kicad_pcb (KiCad board)
At the start: 2 copper layers, 30 x 40 mm, 15 parts, among them J1 Micro_SD_Card, J2 Conn_01x06_MountingPin, U2 AMS1117, U3 74LVC125

Commit message: README doc 18
Parts:
- C1: value C -> 100 nF
Routing:
- added copper zone on F.Cu, net VDD
Other:
- board text added: "0,3000 mm / 0,2000 mm"
- board text added: "HAL SnPb"
- board text removed: "0,2500 mm / 0,2000 mm"
- board text removed: "None"
Changed lines of the file:
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@@
 	(paper "A4")
 	(title_block
-		(title "PCB circuito lector escritor PCB")
+		(title "PCB circuito lector escritor microSD (réplica)")
 		(date "2024-10-09")
 		(rev "Luis Gómez")
-		(company "Fabricante: PCB Chile enlace: https://pcb-chile.cl/")
+		(company "Diseñador. Luis Gómez, hecho en Chile")
+		(comment 1 "versión 0")
+		(comment 2 "Trabajo final curso Diseño Circuitos Impresos, FIUBA")
+		(comment 3 "Fabricante: PCB Chile enlace: https://pcb-chile.cl/")
+		(comment 4 "Licencia: GNU GENERAL PUBLIC LICENSE Version 3, 29 June 2007")
 	)
 	(layers
@@
 			)
 		)
-		(property "Value" "C"
+		(property "Value" "100 nF"
 			(at 0 1.85 0)
 			(layer "F.Fab")
@@
 		)
 	)
-	(gr_text "No"
-		(at 187.764285 45.822 0)
-		(layer "Dwgs.User")
+	(gr_text "Control de impedancia: "
+		(at 222.421423 56.865 0)
+		(layer "User.1")
 		(effects
 			(font
@@
 		)
 	)
-	(gr_text "No"
-		(at 187.764285 49.779 0)
-		(layer "Dwgs.User")
+	(gr_text "Dimensiones generales de la placa: "
+		(at 144.25 48.951 0)
+		(layer "User.1")
 		(effects
 			(font
@@
 		)
 	)
-	(gr_text "Diámetro mínimo de orificio: "
-		(at 221.921423 37.908 0)
-		(layer "Dwgs.User")
+	(gr_text "Número de capas de cobre: "
+		(at 144.25 44.994 0)
+		(layer "User.1")
 		(effects
 			(font
@@
 		)
 	)
-	(gr_text "30,0000 mm x 40,0000 mm"
-		(at 187.764285 33.951 0)
-		(layer "Dwgs.User")
+	(gr_text "HAL SnPb"
+		(at 188.264285 56.865 0)
+		(layer "User.1")
 		(effects
 			(font
@@
 		)
 	)
-	(gr_text "No"
-		(at 260.078565 41.865 0)
-		(layer "Dwgs.User")
+	(gr_text ""
+		(at 260.578565 48.951 0)
+		(layer "User.1")
 		(effects
 			(font
@@
 		)
 	)
-	(gr_text "Pads almena: "
-		(at 143.75 45.822 0)
-		(layer "Dwgs.User")
+	(gr_text "No"
+		(at 188.264285 64.779 0)
+		(layer "User.1")
 		(effects
 			(font
@@
 		)
 	)
-	(gr_text "Número de capas de cobre: "
-		(at 143.75 29.994 0)
-		(layer "Dwgs.User")
+	(gr_text "No"
+		(at 260.578565 56.865 0)
+		(layer "User.1")
 		(effects
 			(font
@@
 		)
 	)
-	(gr_text "Bordes de la placa revestidos: "
-		(at 221.921423 45.822 0)
-		(layer "Dwgs.User")
+	(gr_text "No"
+		(at 260.578565 60.822 0)
+		(layer "User.1")
 		(effects
 			(font
@@
 		)
 	)
-	(gr_text "No"
-		(at 260.078565 45.822 0)
-		(layer "Dwgs.User")
+	(gr_text "Diámetro mínimo de orificio: "
+		(at 222.421423 52.908 0)
+		(layer "User.1")
 		(effects
 			(font
@@
 		)
 	)
-	(gr_text "Dimensiones generales de la placa: "
-		(at 143.75 33.951 0)
-		(layer "Dwgs.User")
+	(gr_text "Pista/espaciado mínimo: "
+		(at 144.25 52.908 0)
+		(layer "User.1")
 		(effects
 			(font
@@
 		)
 	)
-	(gr_text "Pista/espaciado mínimo: "
-		(at 143.75 37.908 0)
-		(layer "Dwgs.User")
+	(gr_text "0,3000 mm"
+		(at 260.578565 52.908 0)
+		(layer "User.1")
 		(effects
 			(font
@@
 		)
 	)
-	(gr_text "Terminación de cobre: "
-		(at 143.75 41.865 0)
-		(layer "Dwgs.User")
+	(gr_text "Bordes de la placa revestidos: "
+		(at 222.421423 60.822 0)
+		(layer "User.1")
 		(effects
 			(font
@@
 		)
 	)
-	(gr_text "Grosor de la placa: "
-		(at 221.921423 29.994 0)
-		(layer "Dwgs.User")
+	(gr_text "30,0000 mm x 40,0000 mm"
+		(at 188.264285 48.951 0)
+		(layer "User.1")
 		(effects
 			(font
@@
 		)
 	)
-	(gr_text "Control de impedancia: "
-		(at 221.921423 41.865 0)
-		(layer "Dwgs.User")
+	(gr_text "1,6000 mm"
+		(at 260.578565 44.994 0)
+		(layer "User.1")
 		(effects
 			(font
@@
 		)
 	)
-	(gr_text "Conectores laterales de tarjeta: "
-		(at 143.75 49.779 0)
-		(layer "Dwgs.User")
+	(gr_text "Línea de seguridad"
+		(at 133 93.5 0)
+		(layer "User.1")
 		(effects
 			(font
-				(size 1.5 1.5)
-				(thickness 0.2)
+				(size 1 1)
+				(thickness 0.15)
 			)
-			(justify left top)
+			(justify left bottom)
 		)
 	)
-	(gr_text "None"
-		(at 187.764285 41.865 0)
-		(layer "Dwgs.User")
+	(gr_text "2"
+		(at 188.264285 44.994 0)
+		(layer "User.1")
 		(effects
 			(font
@@
 		)
 	)
-	(gr_text "CARACTERÍSTICAS DE LA PLACA"
-		(at 143 24.5 0)
-		(layer "Dwgs.User")
+	(gr_text "Terminación de cobre: "
+		(at 144.25 56.865 0)
+		(layer "User.1")
 		(effects
 			(font
-				(size 2 2)
-				(thickness 0.4)
+				(size 1.5 1.5)
+				(thickness 0.2)
 			)
 			(justify left top)
 		)
 	)
-	(gr_text "1,6000 mm"
-		(at 260.078565 29.994 0)
-		(layer "Dwgs.User")
+	(gr_text "Conectores laterales de tarjeta: "
+		(at 144.25 64.779 0)
+		(layer "User.1")
 		(effects
 			(font
@@
 		)
 	)
-	(gr_text "0,3000 mm"
-		(at 260.078565 37.908 0)
-		(layer "Dwgs.User")
+	(gr_text "Grosor de la placa: "
+		(at 222.421423 44.994 0)
+		(layer "User.1")
 		(effects
 			(font
@@
 		)
 	)
-	(gr_text "0,2500 mm / 0,2000 mm"
-		(at 187.764285 37.908 0)
-		(layer "Dwgs.User")
+	(gr_text "Pads almena: "
+		(at 144.25 60.822 0)
+		(layer "User.1")
 		(effects
 			(font
@@
 		)
 	)
-	(gr_text ""
-		(at 260.078565 33.951 0)
-		(layer "Dwgs.User")
+	(gr_text "CARACTERÍSTICAS DE LA PLACA"
+		(at 143.5 39.5 0)
+		(layer "User.1")
 		(effects
 			(font
-				(size 1.5 1.5)
-				(thickness 0.2)
+				(size 2 2)
+				(thickness 0.4)
 			)
 			(justify left top)
 		)
 	)
-	(gr_text "2"
-		(at 187.764285 29.994 0)
-		(layer "Dwgs.User")
+	(gr_text ""
+		(at 222.421423 48.951 0)
+		(layer "User.1")
 		(effects
 			(font
@@
 		)
 	)
-	(gr_text ""
-		(at 221.921423 33.951 0)
-		(layer "Dwgs.User")
+	(gr_text "No"
+		(at 188.264285 60.822 0)
+		(layer "User.1")
 		(effects
 			(font
@@
 		)
 	)
-	(gr_text "Línea de seguridad"
-		(at 133 93.5 0)
+	(gr_text "0,3000 mm / 0,2000 mm"
+		(at 188.264285 52.908 0)
 		(layer "User.1")
 		(effects
 			(font
-				(size 1 1)
-				(thickness 0.15)
+				(size 1.5 1.5)
+				(thickness 0.2)
 			)
-			(justify left bottom)
+			(justify left top)
 		)
 	)
 	(dimension
 		(type aligned)
-		(layer "F.SilkS")
+		(layer "Dwgs.User")
 		(pts
-			(xy 130 140) (xy 130 100)
+			(xy 100 140.16) (xy 130 140.16)
 		)
-		(height 10.7)
-		(gr_text "40,0000 mm"
-			(at 139.6 120 90)
-			(layer "F.SilkS")
+		(height 7.16)
+		(gr_text "30,0000 mm"
+			(at 115 146.17 0)
+			(layer "Dwgs.User")
 			(effects
 				(font
 					(size 1 1)
-					(thickness 0.1)
+					(thickness 0.15)
 				)
 			)
@@
 	(dimension
 		(type aligned)
-		(layer "Dwgs.User")
+		(layer "User.1")
 		(pts
-			(xy 100 140.16) (xy 130 140.16)
+			(xy 130 140) (xy 130 100)
 		)
-		(height 7.16)
-		(gr_text "30,0000 mm"
-			(at 115 146.17 0)
-			(layer "Dwgs.User")
+		(height 10.7)
+		(gr_text "40,0000 mm"
+			(at 139.6 120 90)
+			(layer "User.1")
 			(effects
 				(font
 					(size 1 1)
-					(thickness 0.15)
+					(thickness 0.1)
 				)
 			)
@@
 	)
 	(zone
+		(net 18)
+		(net_name "VDD")
+		(layer "F.Cu")
+		(hatch edge 0.5)
+		(priority 2)
+		(connect_pads
+			(clearance 0.5)
+		)
+		(min_thickness 0.25)
+		(filled_areas_thickness no)
+		(fill yes
+			(thermal_gap 0.5)
+			(thermal_bridge_width 0.5)
+		)
+		(polygon
+			(pts
+				(xy 98.5 110) (xy 109.5 110) (xy 109.5 119) (xy 98.5 119)
+			)
+		)
+	)
+	(zone
 		(net 1)
 		(net_name "GND")
@@
 	)
 	(group "group-boardCharacteristics"
-		(members "123b1b57-1a3f-4eda-9f0d-338e9187de28" "155eb86c-66d5-4e8c-b3e2-c66824216a1d"
-			"1f291698-e700-4b5b-b6a8-785609219514" "2361c5ce-7d9d-4446-8831-beadfe5840ba"
-			"3b09cf38-a0d1-4688-be57-52078ef11f41" "3bb6ebf9-4fc9-401d-9ae5-b2b196775f16"
-			"45f37e39-6129-41da-9e2a-9dda4e447038" "56741f08-d08b-4060-973a-69cbc69b0e97"
-			"7fe631a1-0e08-4c7a-88b9-c481fe87feb2" "8367a6cb-81d9-4471-b18a-943565c84d22"
-			"855f507b-f8c5-4ca2-82d7-ac471d559166" "9713009a-6ca9-4b5e-aea8-37c4d8975b63"
-			"99bd3e82-f963-4271-8cba-5ecd61f0cf85" "a2df6fd9-4674-48d6-9139-8eb8d73b82e0"
-			"ad2b5710-8010-42d9-8936-ffa1da350dbb" "b30c51c4-8984-44ca-8f62-fa5a660c0f67"
-			"b808dd93-9b63-4deb-b3cb-5820f5389681" "bb57831a-5463-4940-9c9d-4cbb4040b9b0"
-			"bc692fe1-44f4-4e18-be45-44fb8ef20be7" "bd0310d1-17b4-40ff-a98c-76fbd8315b4e"
-			"c118ea07-ec2f-481f-9b60-dd3d86203481" "c1dca5a6-c6dc-4ffb-aab6-16bd9a47b0fc"
-			"f72b884e-eb07-482a-b614-1f690b4c1e95"
+		(members "026ef1e3-c7f2-43f3-aef0-27c36d9dd614" "08a2dfd0-c76e-4a97-a2f9-1945dc1da7da"
+			"0fee5705-ff59-409d-81de-1f43e209da0c" "18c15089-9a4c-4239-8565-b844572f028f"
+			"1ce73c3c-04c0-4d24-a4f5-21f8d560c51c" "392b19ed-bea2-4536-a9aa-90a7f580d9e3"
+			"4bfd9a3c-ebb1-4e04-9a21-86440c1bdb31" "507e1d78-aced-4ede-b764-e9b91280aa2c"
+			"5d1067b9-de83-4324-82c4-509ed57b3f33" "76ec77e5-4779-4227-b4ac-fdb23d395b13"
+			"77902fe7-700e-4612-8ba6-b00e7fcbb81f" "7baed1f6-5b3b-4455-8ce2-94fc90bf91b0"
+			"99cdbe05-7b3e-4053-b9e2-8abb56c2f45d" "9a046f7c-362c-4c28-a008-2f217ba6e578"
+			"a0124229-53e5-40f3-8a0d-16585ada9eda" "a58e7ed0-6cdb-4ca4-82f5-928e9554a662"
+			"a71a9e98-0e6b-41b7-8b83-4b22ce0e2b61" "e774c068-48db-48a9-9e0e-6fd8c9cffc00"
+			"ecc585c6-4b83-43c1-9dc3-fc7450eb22d0" "ef6789a3-704f-452b-964d-c98372e0a548"
+			"f436857c-0571-4b0c-ba03-7ddee694b6fe" "f5274e36-b3c1-4f45-b14b-0a24c25a9a8f"
+			"fa573eff-b191-4e06-b8a8-ee18c2de2f45"
 		)
 	)
